File: hardware/OpenLED.kicad_pcb (KiCad board)
At the start: 2 copper layers, 37 x 7 mm, 12 parts, among them J1 5V, J2 GND, J3 DIN, J4 5V, J5 GND, J6 DOUT

Commit message: Prepare OpenLED rev0.1 hardware and panelization
Parts:
- added C3: 100nF, lib:C_0402_1005Metric, F.Cu at (104.7, 104.5)
- added C4: 100nF, lib:C_0402_1005Metric, F.Cu at (111.7, 105.3)
- added C5: 100nF, lib:C_0402_1005Metric, F.Cu at (118.7, 105.3)
- added C6: 100nF, lib:C_0402_1005Metric, F.Cu at (125.7, 105.3)
- added REF**: Tab, lib:Tab, F.Cu at (105.2, 107.0)
- added REF**: Tab, lib:Tab, F.Cu at (105.2, 99.7)
- added REF**: Tab, lib:Tab, F.Cu at (131.8, 107.0)
- added REF**: Tab, lib:Tab, F.Cu at (131.8, 99.7)
- C1, C2: footprint Capacitor_SMD:C_0603_1608Metric -> lib:C_0603_1608Metric
- moved C1 0.78 mm to (103.5, 104.4)
- moved C2 0.18 mm to (132.8, 102.1)
- moved J1 0.07 mm to (101.6, 103.3)
- moved J2 0.07 mm to (101.6, 105.4)
- moved J3 0.07 mm to (101.6, 101.2)
Routing:
- net GND: track 3.26 -> 4.53 mm, vias 10 -> 13
