File: hardware/OpenLED.kicad_sch (KiCad schematic)
At the start: 12 parts, among them J1 5V, J2 GND, J3 DIN, J4 5V, J5 GND, J6 DOUT

Commit message: Prepare OpenLED rev0.1 hardware and panelization
Parts:
- added C3, C4, C5, C6: 100nF, lib:C_0402_1005Metric, symbol Device:C
- C1, C2: footprint Capacitor_SMD:C_0603_1608Metric -> lib:C_0603_1608Metric
Connections:
- net +5V: now also C3.1, C4.1, C5.1, C6.1
- net GND: now also C3.2, C4.2, C5.2, C6.2
Other:
- moved on the sheet: C1, C2
